Commit message: First working version

File: boot0_description/urdf/boot0.xacro (robot description, xacro)
@@ -36,5 +36,5 @@
   <link name="myboat__base">
     <inertial>
-      <mass value="15"/>
+      <mass value="75"/>
       <origin rpy="0 0 0" xyz="-1.0 -0.12 0.1"/>
       <inertia ixx="0.6" ixy="0" ixz="0" iyy="11" iyz="0" izz="11.8"/>
@@ -55,5 +55,5 @@
   <link name="myboat__body">
     <inertial>
-      <mass value="60.0"/>
+      <mass value="1.0"/>
       <origin rpy="0 0 0" xyz="0 0 0.97"/>
       <inertia ixx="19" ixy="0" ixz="0" iyy="19" iyz="0" izz="0.056"/>

Commit message: Set limits on effort

File: boot0_description/urdf/boot0.xacro (robot description, xacro)
@@ -19,5 +19,5 @@
     <origin rpy="-3.13788  0.91639 -3.13874" xyz="-0.03048 -0.03639  2.64237"/>
     <axis xyz="0 1 0"/>
-    <limit effort="10.0" lower="-1.4" upper="1.4" velocity="1.0"/>
+    <limit effort="200.0" lower="-1.4" upper="1.4" velocity="1.0"/>
   </joint>
   <joint name="base_body" type="revolute">

Commit message: nu snap ik commit -a

File: boot0_description/urdf/boot0.xacro (robot description, xacro)
@@ -36,5 +36,5 @@
   <link name="myboat__base">
     <inertial>
-      <mass value="75"/>
+      <mass value="15"/>
       <origin rpy="0 0 0" xyz="-1.0 -0.12 0.1"/>
       <inertia ixx="0.6" ixy="0" ixz="0" iyy="11" iyz="0" izz="11.8"/>
@@ -55,5 +55,5 @@
   <link name="myboat__body">
     <inertial>
-      <mass value="1.0"/>
+      <mass value="60.0"/>
       <origin rpy="0 0 0" xyz="0 0 0.97"/>
       <inertia ixx="19" ixy="0" ixz="0" iyy="19" iyz="0" izz="0.056"/>

Commit message: Added video of instabilities

File: boot0_description/urdf/boot0.xacro (robot description, xacro)
@@ -24,5 +24,5 @@
     <parent link="base_link"/>
     <child link="myboat__body"/>
-    <origin rpy="0.e+00  0.e+00 -4.e-05" xyz="-0.98209 -0.1049   0.15209"/>
+    <origin rpy="0.e+00  0.e+00 -4.e-05" xyz="-0.1 -0.1   0.15209"/>
     <axis xyz="0 1 0"/>
     <limit effort="2000.0" lower="-1.4" upper="1.4" velocity="1.0"/>
@@ -37,17 +37,17 @@
     <inertial>
       <mass value="15"/>
-      <origin rpy="0 0 0" xyz="-1.0 -0.12 0.1"/>
+      <origin rpy="0 0 0" xyz="0.0 0.0 0.1"/>
       <inertia ixx="0.6" ixy="0" ixz="0" iyy="11" iyz="0" izz="11.8"/>
     </inertial>
     <collision>
-      <origin rpy="0 0 0" xyz="-1.0 -0.12   0.1"/>
+      <origin rpy="0 0 0" xyz="0.0 0.0   0.1"/>
       <geometry>
-        <box size="3.0 0.663318 0.197068"/>
+        <box size="3.0 0.7 0.2"/>
       </geometry>
     </collision>
     <visual>
-      <origin rpy="0 0 0" xyz="-1.06112 -0.1246   0.1"/>
+      <origin rpy="0 0 0" xyz="0.0 0.0  0.1"/>
       <geometry>
-        <box size="3.0 0.663318 0.197068"/>
+        <box size="3.0 0.7 0.2"/>
       </geometry>
     </visual>

File: boot1_description/urdf/boot1.xacro (robot description, xacro)
@@ -2,29 +2,49 @@
 <robot name="myboat"  xmlns:xacro="http://www.ros.org/wiki/xacro">
   <!-- Constants for robot dimensions -->
-  <xacro:property name="PI" value="3.1415926535897931"/>
   <!-- Import all Gazebo-customization elements, including Gazebo colors -->
   <xacro:include filename="$(find boot1_description)/urdf/boot1.gazebo" />
   <!-- Import Rviz colors -->
   <xacro:include filename="$(find boot1_description)/urdf/materials.xacro" />
-  <joint name="body_arm" type="revolute">
-    <parent link="myboat__body"/>
-    <child link="myboat__arm"/>
-    <origin rpy="-1.45000e-03 -1.54681e+00  3.75000e-03" xyz="0.02714 -0.00665  1.9954"/>
-    <axis xyz="0 1 0"/>
-    <limit effort="200.0" lower="-1.4" upper="1.4" velocity="1.0"/>
-  </joint>
-  <joint name="arm_blad" type="revolute">
-    <parent link="myboat__arm"/>
-    <child link="myboat__blad"/>
-    <origin rpy="-3.13788  0.91639 -3.13874" xyz="-0.03048 -0.03639  2.64237"/>
-    <axis xyz="0 1 0"/>
-    <limit effort="200.0" lower="-1.4" upper="1.4" velocity="1.0"/>
-  </joint>
-  <joint name="base_body" type="revolute">
-    <parent link="base_link"/>
-    <child link="myboat__body"/>
-    <origin rpy="0.e+00  0.e+00 -4.e-05" xyz="-0.98209 -0.1049   0.15209"/>
-    <axis xyz="0 1 0"/>
-    <limit effort="2000.0" lower="-1.4" upper="1.4" velocity="1.0"/>
+  <joint name="starboard_rowlock_joint" type="revolute">
+    <parent link="skiff"/>
+    <child link="starboard_rowlock"/>
+    <origin rpy="0.0  0.0 0.0" xyz="0.0 0.8 0.32"/>
+    <axis xyz="0 0 1"/>
+    <limit effort="300.0" lower="-1.4" upper="1.4" velocity="1.0"/>
+  </joint>
+  <joint name="port_rowlock_joint" type="revolute">
+    <parent link="skiff"/>
+    <child link="port_rowlock"/>
+    <origin rpy="0.0  0.0 0.0" xyz="0.0 -0.8 0.3"/>
+    <axis xyz="0 0 1"/>
+    <limit effort="300.0" lower="-1.4" upper="1.4" velocity="1.0"/>
+  </joint>
+  <joint name="starboard_rowlock_oar_joint" type="revolute">
+    <parent link="starboard_rowlock"/>
+    <child link="starboard_oar"/>
+    <origin rpy="0.0  ${pi/2} -${pi/2}" xyz="0.0 0.0   0.02"/>
+    <axis xyz="0 1 0"/>
+    <limit effort="2000.0" lower="-0.4" upper="0.0" velocity="1.0"/>
+  </joint>
+  <joint name="port_rowlock_oar_joint" type="revolute">
+    <parent link="port_rowlock"/>
+    <child link="port_oar"/>
+    <origin rpy="0.0  ${pi/2} -${pi/2}" xyz="0.0 0.0   0.02"/>
+    <axis xyz="0 1 0"/>
+    <limit effort="2000.0" lower="0.0" upper="0.4" velocity="1.0"/>
+  </joint>
+  <joint name="starboard_blade_joint" type="revolute">
+    <parent link="starboard_oar"/>
+    <child link="starboard_blade"/>
+    <origin rpy="0 0  0.0" xyz="0.0 0.0   -1.8"/>
+    <axis xyz="0 1 0"/>
+    <limit effort="1000.0" lower="-0.2" upper="0.2" velocity="1.0"/>
+  </joint>
+  <joint name="port_blade_joint" type="revolute">
+    <parent link="port_oar"/>
+    <child link="port_blade"/>
+    <origin rpy="0.0  0 0.0" xyz="0.0 0.0   1.8"/>
+    <axis xyz="0 1 0"/>
+    <limit effort="1000.0" lower="-0.2" upper="0.2" velocity="1.0"/>
   </joint>
   <link name="base_link"/>
@@ -32,79 +52,138 @@
   <joint name="dummy" type="fixed">
     <parent link="base_link"/>
-    <child link="myboat__base"/>
-  </joint>
-  <link name="myboat__base">
-    <inertial>
-      <mass value="15"/>
-      <origin rpy="0 0 0" xyz="-1.0 -0.12 0.1"/>
-      <inertia ixx="0.6" ixy="0" ixz="0" iyy="11" iyz="0" izz="11.8"/>
-    </inertial>
-    <collision>
-      <origin rpy="0 0 0" xyz="-1.0 -0.12   0.1"/>
-      <geometry>
-        <box size="3.0 0.663318 0.197068"/>
-      </geometry>
-    </collision>
-    <visual>
-      <origin rpy="0 0 0" xyz="-1.06112 -0.1246   0.1"/>
-      <geometry>
-        <box size="3.0 0.663318 0.197068"/>
-      </geometry>
-    </visual>
-  </link>
-  <link name="myboat__body">
-    <inertial>
-      <mass value="60.0"/>
-      <origin rpy="0 0 0" xyz="0 0 0.97"/>
-      <inertia ixx="19" ixy="0" ixz="0" iyy="19" iyz="0" izz="0.056"/>
-    </inertial>
-    <collision>
-      <origin rpy="0 0 0" xyz="0   0   0.97"/>
-      <geometry>
-        <box size="0.100516 0.036549 1.95488"/>
-      </geometry>
-    </collision>
-    <visual>
-      <origin rpy="0 0 0" xyz="0   0   0.97"/>
-      <geometry>
-        <box size="0.100516 0.036549 1.95488"/>
-      </geometry>
-    </visual>
-  </link>
-  <link name="myboat__blad">
-    <inertial>
-      <mass value="1.0"/>
-      <origin rpy="0 0 0" xyz="0 0 -0.05"/>
+    <child link="skiff"/>
+  </joint>
+  <link name="skiff">
+    <inertial>
+      <mass value="75"/>   <!-- 15 + 60 voor de roeier -->
+      <origin rpy="0 0 0" xyz="0.0 0.0 0.1"/>
+      <inertia ixx="3.2" ixy="0" ixz="0" iyy="54.2" iyz="0" izz="57"/>
+<!--      <inertia ixx="0.6" ixy="0" ixz="0" iyy="11" iyz="0" izz="11.8"/>  -->
+    </inertial>
+    <collision>
+      <origin rpy="0 0 0" xyz="0.0 0.0   0.1"/>
+      <geometry>
+        <box size="3.0 0.7 0.2"/>
+      </geometry>
+    </collision>
+    <visual>
+      <!-- should be a nice skull shape including riggers-->
+      <origin rpy="0 0 0" xyz="0.0 0.0   0.1"/>
+      <geometry>
+        <box size="3.0 0.7 0.2"/>
+      </geometry>
+    </visual>
+  </link>
+  <link name="starboard_rowlock">
+    <inertial>
+      <mass value="0.1"/>
+      <origin rpy="0 0 0" xyz="0.0 0.0 0.0"/>
+      <inertia ixx="0.00007" ixy="0" ixz="0" iyy="0.00007" iyz="0" izz="0.000007"/>
+    </inertial>
+    <collision>
+      <origin rpy="0 0 0" xyz="0.0 0.0   0.0"/>
+      <geometry>
+        <box size="0.02 0.02 0.04"/>
+      </geometry>
+    </collision>
+    <visual>
+      <origin rpy="0 0 0" xyz="0.0 0.0   0.0"/>
+      <geometry>
+        <box size="0.02 0.02 0.04"/>
+      </geometry>
+    </visual>
+  </link>
+  <link name="port_rowlock">
+    <inertial>
+      <mass value="0.1"/>
+      <origin rpy="0 0 0" xyz="0.0 0.0 0.0"/>
+      <inertia ixx="0.00007" ixy="0" ixz="0" iyy="0.00007" iyz="0" izz="0.000007"/>
+    </inertial>
+    <collision>
+      <origin rpy="0 0 0" xyz="0.0 0.0   0.0"/>
+      <geometry>
+        <box size="0.02 0.02 0.04"/>
+      </geometry>
+    </collision>
+    <visual>
+      <origin rpy="0 0 0" xyz="0.0 0.0   0.0"/>
+      <geometry>
+        <box size="0.02 0.02 0.04"/>
+      </geometry>
+    </visual>
+  </link>
+  <link name="starboard_oar">
+    <inertial>
+      <mass value="1.0"/>
+      <origin rpy="0 0 0" xyz="0 0 -0.45"/>
+      <inertia ixx="0.6" ixy="0" ixz="0" iyy="0.6" iyz="0" izz="0.001"/>
+    </inertial>
+    <collision>
+      <origin rpy="0 0 0" xyz="0   0   -0.45"/>
+      <geometry>
+        <cylinder length="2.7" radius="0.02"/>
+      </geometry>
+    </collision>
+    <visual>
+      <origin rpy="0 0 0" xyz="0   0.0   -0.45"/>
+      <geometry>
+        <cylinder length="2.7" radius="0.02"/>
+      </geometry>
+    </visual>
+  </link>
+  <link name="port_oar">
+    <inertial>
+      <mass value="1.0"/>
+      <origin rpy="0 0 0" xyz="0 0 0.45"/>
+      <inertia ixx="0.6" ixy="0" ixz="0" iyy="0.6" iyz="0" izz="0.001"/>
+    </inertial>
+    <collision>
+      <origin rpy="0 0 0" xyz="0   0   0.45"/>
+      <geometry>
+        <cylinder length="2.7" radius="0.02"/>  <!-- 2.0 to prevent collissions  -->
+      </geometry>
+    </collision>
+    <visual>
+      <origin rpy="0 0 0" xyz="0   0   0.45"/>
+      <geometry>
+        <cylinder length="2.7" radius="0.02"/>
+      </geometry>
+    </visual>
+  </link>
+  <link name="starboard_blade">
+    <inertial>
+      <mass value="1.0"/>
+      <origin rpy="0 -1.4 0" xyz="0.02 0 -0.02"/>
       <inertia ixx="0.34" ixy="0" ixz="0" iyy="0.34" iyz="0" izz="0.73"/>
     </inertial>
     <collision>
-      <origin rpy="0 0 0" xyz="0    0   -0.05"/>
-      <geometry>
-        <box size="0.695693 0.648073 0.108244"/>
-      </geometry>
-    </collision>
-    <visual>
-      <origin rpy="0 0 0" xyz="0    0   -0.05"/>
-      <geometry>
-        <box size="0.695693 0.648073 0.108244"/>
-      </geometry>
-    </visual>
-  </link>
-  <link name="myboat__arm">
-    <inertial>
-      <mass value="1.0"/>
-      <origin rpy="0 0 0" xyz="0 0 1.3"/>
-      <inertia ixx="0.32" ixy="0" ixz="0" iyy="0.32" iyz="0" izz="0.0016"/>
-    </inertial>
-    <collision>
-      <origin rpy="0 0 0" xyz="0  0  1.3"/>
-      <geometry>
-        <cylinder length="1.97792" radius="0.05655"/>
-      </geometry>
-    </collision>
-    <visual>
-      <origin rpy="0 0 0" xyz="0  0  1.3"/>
-      <geometry>
-        <cylinder length="2.5" radius="0.05655"/>
+      <origin rpy="0 -1.4 0" xyz="0.02    0   -0.02"/>
+      <geometry>
+        <box size="0.2 0.1 0.03"/>
+      </geometry>
+    </collision>
+    <visual>
+      <origin rpy="0 -1.4 0" xyz="0.02    0   -0.02"/>
+      <geometry>
+        <box size="0.2 0.1 0.03"/>
+      </geometry>
+    </visual>
+  </link>
+  <link name="port_blade">
+    <inertial>
+      <mass value="1.0"/>
+      <origin rpy="0 1.4 0" xyz="0.02 0 -0.02"/>
+      <inertia ixx="0.34" ixy="0" ixz="0" iyy="0.34" iyz="0" izz="0.73"/>
+    </inertial>
+    <collision>
+      <origin rpy="0 1.4 0" xyz="0.02    0   -0.02"/>
+      <geometry>
+        <box size="0.2 0.1 0.03"/>
+      </geometry>
+    </collision>
+    <visual>
+      <origin rpy="0 1.4 0" xyz="0.02    0.0  -0.02"/>
+      <geometry>
+        <box size="0.2 0.1 0.03"/>
       </geometry>
     </visual>
@@ -112,5 +191,5 @@
   <transmission name="tran1">
     <type>transmission_interface/SimpleTransmission</type>
-    <joint name="base_body">
+    <joint name="starboard_rowlock_joint">
       <hardwareInterface>hardware_interface/EffortJointInterface</hardwareInterface>
     </joint>
@@ -121,5 +200,5 @@
   <transmission name="tran2">
     <type>transmission_interface/SimpleTransmission</type>
-    <joint name="body_arm">
+    <joint name="port_rowlock_joint">
       <hardwareInterface>hardware_interface/EffortJointInterface</hardwareInterface>
     </joint>
@@ -130,8 +209,35 @@
   <transmission name="tran3">
     <type>transmission_interface/SimpleTransmission</type>
-    <joint name="arm_blad">
-      <hardwareInterface>hardware_interface/EffortJointInterface</hardwareInterface>
-    </joint>
-    <actuator name="motor2">
+    <joint name="starboard_rowlock_oar_joint">
+      <hardwareInterface>hardware_interface/EffortJointInterface</hardwareInterface>
+    </joint>
+    <actuator name="motor3">
+      <mechanicalReduction>1</mechanicalReduction>
+    </actuator>
+  </transmission>
+  <transmission name="tran4">
+    <type>transmission_interface/SimpleTransmission</type>
+    <joint name="port_rowlock_oar_joint">
+      <hardwareInterface>hardware_interface/EffortJointInterface</hardwareInterface>
+    </joint>
+    <actuator name="motor4">
+      <mechanicalReduction>1</mechanicalReduction>
+    </actuator>
+  </transmission>
+  <transmission name="tran5">
+    <type>transmission_interface/SimpleTransmission</type>
+    <joint name="starboard_blade_joint">
+      <hardwareInterface>hardware_interface/EffortJointInterface</hardwareInterface>
+    </joint>
+    <actuator name="motor5">
+      <mechanicalReduction>1</mechanicalReduction>
+    </actuator>
+  </transmission>
+  <transmission name="tran6">
+    <type>transmission_interface/SimpleTransmission</type>
+    <joint name="port_blade_joint">
+      <hardwareInterface>hardware_interface/EffortJointInterface</hardwareInterface>
+    </joint>
+    <actuator name="motor6">
       <mechanicalReduction>1</mechanicalReduction>
     </actuator>
